Commit message: new building with pointcloud fixed

File: src/description/urdf/robot_core.xacro (robot description, xacro)
@@ -24,34 +24,34 @@
 </joint>
 <link name="building">
-<visual>
-    <origin xyz="0 -40.030 0" rpy="0 0 ${PI/2}"/>
-    <geometry>
-        <mesh filename="package://description/meshes/building.stl" scale="0.5 0.5 0.5"/>
-    </geometry>
-    <material name="black"/>
-</visual>
-<collision>
-    <origin xyz="0 -40.030 0" rpy="0 0 ${PI/2}"/>
-    <geometry>
-        <mesh filename="package://description/meshes/building.stl" scale="0.5 0.5 0.5"/>
-    </geometry>
-    <surface>
-        <friction>
-          <ode>
-            <mu>20</mu>
-            <mu2>20</mu2>
-          </ode>
-        </friction>
-      </surface>
-</collision>
-<inertial>
-    <origin xyz="0 -40.030 0" rpy="0 0 ${PI/2}"/>
-    <mass value="5000"/>
-    <inertia
-            ixx="100.0" ixy="0.0" ixz="0.0"
-            iyy="100.0" iyz="0.0"
-            izz="100.0"/>
-</inertial>
-</link>
+    <visual>
+        <origin xyz="0 0 0" rpy="0 0 0"/>
+        <geometry>
+            <mesh filename="package://description/meshes/building7_f.stl" scale="1 1 1"/>
+        </geometry>
+        <material name="orange"/>
+    </visual>
+    <collision>
+        <origin xyz="0 0 0" rpy="0 0 0"/>
+        <geometry>
+            <mesh filename="package://description/meshes/building7_f.stl" scale="1 1 1"/>
+        </geometry>
+        <surface>
+            <friction>
+              <ode>
+                <mu>20</mu>
+                <mu2>20</mu2>
+              </ode>
+            </friction>
+          </surface>
+    </collision>
+    <inertial>
+        <origin xyz="0 0 0" rpy="0 0 0"/>
+        <mass value="5000"/>
+        <inertia
+                ixx="100.0" ixy="0.0" ixz="0.0"
+                iyy="100.0" iyz="0.0"
+                izz="100.0"/>
+    </inertial>
+    </link>
     <!--BASE OF THE PTZ CAMERA-->
     <joint name="base_joint" type="fixed">
@@ -62,5 +62,5 @@
     <link name="base_ptz_camera_link">
         <visual>
-            <origin xyz="0 20 0" rpy="0 0 0"/>
+            <origin xyz="0 0 0" rpy="0 0 0"/>
             <geometry>
                 <!--box size="0.07 0.11 0.02"/-->
@@ -70,5 +70,5 @@
         </visual>
         <collision>
-            <origin xyz="0 20 0" rpy="0 0 0"/>
+            <origin xyz="0 0 0" rpy="0 0 0"/>
             <geometry>
                 <mesh filename="package://description/meshes/base.stl" scale="0.001 0.001 0.001"/>
@@ -76,5 +76,5 @@
         </collision>
         <inertial>
-            <origin xyz="0 20 0" rpy="0 0 0"/>
+            <origin xyz="0 0 0" rpy="0 0 0"/>
             <mass value="1"/>
             <inertia
